File: files/kicad/RunType58/RunType58.kicad_sch (KiCad schematic)
At the start: 140 parts, among them SW1 SW_PUSH, SW10 SW_PUSH, SW11 SW_PUSH, SW12 SW_PUSH, SW13 SW_PUSH, SW14 SW_PUSH, SW15 SW_PUSH, SW16 SW_PUSH, SW17 SW_PUSH, SW18 SW_PUSH, SW19 SW_PUSH, SW2 SW_PUSH, SW20 SW_PUSH, SW21 SW_PUSH, SW22 SW_PUSH, SW23 SW_PUSH, SW24 SW_PUSH, SW25 SW_PUSH, SW26 SW_PUSH, SW27 SW_PUSH, SW28 SW_PUSH, SW29 SW_PUSH, SW3 SW_PUSH, SW30 SW_PUSH, SW31 SW_PUSH, SW32 SW_PUSH, SW33 SW_PUSH, SW34 SW_PUSH, SW35 SW_PUSH, SW36 SW_PUSH, SW37 SW_PUSH, SW38 SW_PUSH, SW39 SW_PUSH, SW4 SW_PUSH, SW40 SW_PUSH, SW41 SW_PUSH, SW42 SW_PUSH, SW43 SW_PUSH, SW44 SW_PUSH, SW45 SW_PUSH, SW46 SW_PUSH, SW47 SW_PUSH, SW48 SW_PUSH, SW49 SW_PUSH, SW5 SW_PUSH, SW50 SW_PUSH, SW51 SW_PUSH, SW52 SW_PUSH, SW53 SW_PUSH, SW54 SW_PUSH, SW55 SW_PUSH, SW56 SW_PUSH, SW57 SW_PUSH, SW58 SW_PUSH, SW6 SW_PUSH, SW7 SW_PUSH, SW8 SW_PUSH, SW9 SW_PUSH, U1 nice_nano, U2 nice_nano

Commit message: gathering some of the updates
Connections:
- net ROWL3: now also D52.1 (K)
- net ROWL4: no longer D52.1 (K)
Changed lines of the file:
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@@
   (junction (at 173.99 205.74) (diameter 0) (color 0 0 0 0)
   )
+  (junction (at 273.05 212.09) (diameter 0) (color 0 0 0 0)
+  )
   (junction (at 119.38 73.66) (diameter 0) (color 0 0 0 0)
   )
@@
   )
   (junction (at 167.64 39.37) (diameter 0) (color 0 0 0 0)
-  )
-  (junction (at 295.91 229.87) (diameter 0) (color 0 0 0 0)
   )
   (junction (at 213.36 180.34) (diameter 0) (color 0 0 0 0)
@@
     (stroke (width 0) (type default) (color 0 0 0 0))
   )
-  (wire (pts (xy 295.91 229.87) (xy 298.45 229.87))
-    (stroke (width 0) (type default) (color 0 0 0 0))
-  )
   (wire (pts (xy 167.64 36.83) (xy 167.64 39.37))
     (stroke (width 0) (type default) (color 0 0 0 0))
@@
     (stroke (width 0) (type default) (color 0 0 0 0))
   )
-  (wire (pts (xy 298.45 212.09) (xy 298.45 229.87))
-    (stroke (width 0) (type default) (color 0 0 0 0))
-  )
   (wire (pts (xy 187.96 36.83) (xy 189.23 36.83))
     (stroke (width 0) (type default) (color 0 0 0 0))
@@
     (stroke (width 0) (type default) (color 0 0 0 0))
   )
+  (wire (pts (xy 273.05 212.09) (xy 298.45 212.09))
+    (stroke (width 0) (type default) (color 0 0 0 0))
+  )
